File: NSP2D.brd (EAGLE design)
At the start: 49.2 x 82 mm, 21 parts, among them Q1 600mA/40V, Q2 IRF540

Commit message: Added missing pullup resistors to SCL SDA for I2C bus
Parts:
- added R6, R7: 4.5k, SparkFun-Passives:1/6W-RES
Connections:
- net SCL: now also R7.2
- net SDA: now also R6.2
- net V_BATT: now also R6.1, R7.1
Routing:
- net V_BATT: track 107.6 -> 130.3 mm
- net SDA: track 21.5 -> 23.6 mm
- net UART4_TX: track 19.0 -> 17.6 mm
- net SCL: track 21.6 -> 20.4 mm
- net UART4_RX: track 18.3 -> 17.6 mm
Changed lines of the file:
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@@
 <element name="R4" library="SparkFun-Passives" package="1/6W-RES" value="1K" x="35.56" y="57.15" rot="R270"/>
 <element name="LED3" library="SparkFun-Connectors" package="1X02" value="" x="44.45" y="54.61" rot="R180"/>
+<element name="R6" library="SparkFun-Passives" package="1/6W-RES" value="4.5k" x="31.75" y="45.72"/>
+<element name="R7" library="SparkFun-Passives" package="1/6W-RES" value="4.5k" x="31.75" y="41.91"/>
 </elements>
 <signals>
@@
 <wire x1="46.99" y1="49.53" x2="44.45" y2="49.53" width="0.8128" layer="16"/>
 <wire x1="44.45" y1="49.53" x2="44.45" y2="45.72" width="0.8128" layer="16"/>
-<wire x1="44.45" y1="45.72" x2="44.45" y2="41.91" width="0.8128" layer="16"/>
+<wire x1="44.45" y1="41.91" x2="44.45" y2="45.72" width="0.8128" layer="16"/>
 <wire x1="44.45" y1="41.91" x2="44.45" y2="36.195" width="0.8128" layer="16"/>
 <wire x1="44.45" y1="36.195" x2="45.085" y2="36.195" width="0.3048" layer="16"/>
@@
 <wire x1="44.45" y1="24.13" x2="39.37" y2="24.13" width="0.8128" layer="16"/>
 <wire x1="39.37" y1="24.13" x2="39.37" y2="26.67" width="0.8128" layer="16"/>
+<contactref element="R6" pad="1"/>
+<contactref element="R7" pad="1"/>
+<wire x1="29.25" y1="41.91" x2="29.25" y2="45.72" width="0.3048" layer="1"/>
+<wire x1="29.25" y1="45.72" x2="29.25" y2="47.411" width="0.3048" layer="1"/>
+<wire x1="29.25" y1="47.411" x2="29.337" y2="47.498" width="0.3048" layer="1"/>
+<wire x1="29.337" y1="47.498" x2="44.577" y2="47.498" width="0.3048" layer="1"/>
+<wire x1="44.577" y1="47.498" x2="44.577" y2="45.847" width="0.3048" layer="1"/>
+<wire x1="44.577" y1="45.847" x2="44.45" y2="45.72" width="0.3048" layer="1"/>
 </signal>
 <signal name="UART5_RX">
@@
 <contactref element="I2CX" pad="2"/>
 <contactref element="MCU" pad="24"/>
-<wire x1="39.37" y1="49.53" x2="39.37" y2="45.72" width="0.3048" layer="16"/>
-<wire x1="39.37" y1="43.815" x2="30.607" y2="43.815" width="0.3048" layer="1"/>
-<wire x1="30.607" y1="43.815" x2="30.48" y2="43.688" width="0.3048" layer="1"/>
-<wire x1="30.48" y1="43.688" x2="30.48" y2="40.64" width="0.3048" layer="1"/>
-<wire x1="30.48" y1="40.64" x2="26.67" y2="40.64" width="0.3048" layer="1"/>
-<wire x1="39.37" y1="45.72" x2="39.37" y2="43.815" width="0.3048" layer="1"/>
+<wire x1="39.37" y1="45.72" x2="39.37" y2="49.53" width="0.3048" layer="16"/>
+<contactref element="R6" pad="2"/>
+<wire x1="34.25" y1="45.72" x2="34.29" y2="45.68" width="0.3048" layer="16"/>
+<wire x1="34.29" y1="45.68" x2="34.29" y2="43.688" width="0.3048" layer="16"/>
+<wire x1="34.29" y1="43.688" x2="39.37" y2="43.688" width="0.3048" layer="16"/>
+<wire x1="39.37" y1="43.688" x2="39.37" y2="45.72" width="0.3048" layer="16"/>
+<wire x1="34.29" y1="43.688" x2="31.75" y2="43.688" width="0.3048" layer="16"/>
+<wire x1="31.75" y1="43.688" x2="31.75" y2="40.64" width="0.3048" layer="16"/>
+<wire x1="31.75" y1="40.64" x2="26.67" y2="40.64" width="0.3048" layer="16"/>
 </signal>
 <signal name="UART4_RX">
 <contactref element="MCU" pad="21"/>
 <contactref element="LOGR" pad="1"/>
-<wire x1="36.83" y1="41.91" x2="31.75" y2="41.91" width="0.3048" layer="16"/>
-<wire x1="31.75" y1="41.91" x2="31.75" y2="34.29" width="0.3048" layer="16"/>
 <wire x1="27.94" y1="34.29" x2="26.67" y2="33.02" width="0.3048" layer="16"/>
-<wire x1="31.75" y1="34.29" x2="27.94" y2="34.29" width="0.3048" layer="16"/>
+<wire x1="27.94" y1="34.29" x2="31.75" y2="34.29" width="0.3048" layer="16"/>
+<wire x1="31.75" y1="34.29" x2="31.75" y2="36.83" width="0.3048" layer="16"/>
+<wire x1="31.75" y1="36.83" x2="33.02" y2="38.1" width="0.3048" layer="16"/>
+<wire x1="33.02" y1="38.1" x2="36.83" y2="38.1" width="0.3048" layer="16"/>
+<wire x1="36.83" y1="38.1" x2="36.83" y2="41.91" width="0.3048" layer="16"/>
 </signal>
 <signal name="UART4_TX">
 <contactref element="MCU" pad="22"/>
 <contactref element="LOGR" pad="2"/>
+<wire x1="39.37" y1="41.91" x2="39.37" y2="39.37" width="0.3048" layer="1"/>
+<wire x1="39.37" y1="39.37" x2="33.02" y2="39.37" width="0.3048" layer="1"/>
+<wire x1="33.02" y1="39.37" x2="30.48" y2="36.83" width="0.3048" layer="1"/>
+<wire x1="30.48" y1="36.83" x2="30.48" y2="35.56" width="0.3048" layer="1"/>
 <wire x1="30.48" y1="35.56" x2="26.67" y2="35.56" width="0.3048" layer="1"/>
-<wire x1="39.37" y1="41.91" x2="39.37" y2="39.37" width="0.3048" layer="1"/>
-<wire x1="39.37" y1="39.37" x2="30.48" y2="39.37" width="0.3048" layer="1"/>
-<wire x1="30.48" y1="39.37" x2="30.48" y2="35.56" width="0.3048" layer="1"/>
 </signal>
 <signal name="N$6">
@@
 <contactref element="MCU" pad="23"/>
 <wire x1="36.83" y1="49.53" x2="36.83" y2="45.72" width="0.3048" layer="16"/>
-<wire x1="36.83" y1="45.72" x2="30.48" y2="45.72" width="0.3048" layer="16"/>
-<wire x1="30.48" y1="45.72" x2="30.48" y2="38.1" width="0.3048" layer="16"/>
-<wire x1="30.48" y1="38.1" x2="26.67" y2="38.1" width="0.3048" layer="16"/>
+<contactref element="R7" pad="2"/>
+<wire x1="34.25" y1="43.648" x2="34.25" y2="41.91" width="0.3048" layer="1"/>
+<wire x1="34.25" y1="43.648" x2="34.29" y2="43.688" width="0.3048" layer="1"/>
+<wire x1="34.29" y1="43.688" x2="36.83" y2="43.688" width="0.3048" layer="1"/>
+<wire x1="36.83" y1="43.688" x2="36.83" y2="45.72" width="0.3048" layer="1"/>
+<wire x1="34.25" y1="41.91" x2="34.25" y2="40.092" width="0.3048" layer="1"/>
+<wire x1="31.10341875" y1="38.1" x2="26.67" y2="38.1" width="0.3048" layer="1"/>
+<wire x1="33.9852" y1="39.8272" x2="32.83061875" y2="39.8272" width="0.3048" layer="1"/>
+<wire x1="32.83061875" y1="39.8272" x2="31.10341875" y2="38.1" width="0.3048" layer="1"/>
+<wire x1="34.25" y1="40.092" x2="33.9852" y2="39.8272" width="0.3048" layer="1"/>
 </signal>
 <signal name="N$2">

Commit message: Added capacitor for batt source
Parts:
- added C1: 1mF, SparkFun-Capacitors:CPOL-RADIAL-5MM-10MM
- renumbered I2CX to I2C, I2CX1 to I2C1
Connections:
- net 3.3V: now also R6.1, R7.1
- net GND: now also C1.-
- net V_BATT: now also C1.+; no longer R6.1, R7.1
Routing:
- net N$5: track 31.8 -> 19.3 mm
- net V_BATT: track 130.3 -> 119.6 mm
- net 3.3V: track 0.00 -> 3.81 mm
- net N$2: track 59.7 -> 56.6 mm
- net SDA: track 23.6 -> 26.0 mm
Other:
- board size 49.2 x 82 mm -> 49.2 x 88.4 mm
- board text added: "Designed & Built in Mexico @ ASFM STEM LAB"
- board text added: "FLIGHT COMPUTER"
- board text added: "HLM1"
- board text added: "Rev 1.0 - OCT 2017"
- board text removed: "Designed + Built in Mexico @ ASFM"
- board text removed: "HLM STEM LAB TECH"
- board text removed: "Oct 2017 | NSP @ ASFM | HLM 1 FLIGHT CTL"

Commit message: Finished R1 for manufacturing
Other:
- board size 49.2 x 88.4 mm -> 51.1 x 89.4 mm
- board text added: "+"
- board text added: "-"
- board text added: "ANT CLIP"
- board text added: "BAT"
- board text added: "BUZR"
- board text added: "GPS"
- board text added: "HEAT"
- board text added: "I2C NET"
- board text added: "LEDS"
- board text added: "LOGR"
- board text added: "SAT"
- board text added: "TEMP"
- board text added: "http://github.com/asfm-hlm-stemlab"
- board text removed: "ANT LOCK"
Changed lines of the file:
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@@
 <board>
 <plain>
-<wire x1="0" y1="15.24" x2="49.2" y2="15.24" width="1" layer="20"/>
-<wire x1="49.2" y1="15.24" x2="49.2" y2="90.668" width="1" layer="20"/>
-<wire x1="49.2" y1="90.668" x2="0" y2="90.668" width="1" layer="20"/>
+<wire x1="0" y1="15.24" x2="51.105" y2="15.24" width="1" layer="20"/>
+<wire x1="51.105" y1="15.24" x2="51.105" y2="90.668" width="1" layer="20"/>
+<wire x1="51.105" y1="90.668" x2="0" y2="90.668" width="1" layer="20"/>
 <wire x1="0" y1="90.668" x2="0" y2="15.24" width="1" layer="20"/>
-<text x="20.32" y="74.93" size="3.81" layer="26" rot="MR270">ASFM | HLM 1 | v1.0</text>
-<text x="11.938" y="81.026" size="1.27" layer="25">FLIGHT COMPUTER</text>
-<polygon width="0.8128" layer="20">
-<vertex x="39.116" y="15.113"/>
-<vertex x="39.116" y="2.413"/>
-<vertex x="8.382" y="2.286"/>
-<vertex x="8.382" y="14.986"/>
+<text x="20.32" y="74.93" size="3.81" layer="22" rot="MR270">ASFM | HLM 1 | v1.0</text>
+<text x="10.922" y="81.026" size="1.27" layer="21">FLIGHT COMPUTER</text>
+<text x="5.08" y="23.241" size="2" layer="21" rot="R90">Designed &amp; Built in Mexico @ ASFM STEM LAB</text>
+<text x="7.493" y="17.653" size="1.9304" layer="21">Rev 1.0 - OCT 2017</text>
+<text x="11.049" y="83.058" size="5.08" layer="21">HLM1</text>
+<polygon width="0.3048" layer="20">
+<vertex x="6.35" y="15.24"/>
+<vertex x="6.35" y="1.27"/>
+<vertex x="35.56" y="1.27"/>
+<vertex x="39.37" y="5.08"/>
+<vertex x="39.37" y="15.24"/>
 </polygon>
-<hole x="10.16" y="11.43" drill="2"/>
-<hole x="10.16" y="6.35" drill="2"/>
-<hole x="19.05" y="11.43" drill="2"/>
-<hole x="19.05" y="6.35" drill="2"/>
-<text x="11.43" y="7.112" size="1.778" layer="25"> ANT
-LOCK</text>
-<text x="5.08" y="23.241" size="2" layer="25" rot="R90">Designed &amp; Built in Mexico @ ASFM STEM LAB</text>
-<text x="7.747" y="16.637" size="1.9304" layer="25">Rev 1.0 - OCT 2017</text>
-<text x="11.049" y="83.058" size="5.08" layer="25">HLM1</text>
+<hole x="21.59" y="12.7" drill="4"/>
+<hole x="21.59" y="5.08" drill="4"/>
+<hole x="10.16" y="5.08" drill="4"/>
+<hole x="10.16" y="12.7" drill="4"/>
+<text x="13.208" y="6.985" size="1.9304" layer="21">ANT
+CLIP</text>
+<text x="46.228" y="66.802" size="1.016" layer="21">GPS</text>
+<text x="46.228" y="72.009" size="1.016" layer="21">BUZR</text>
+<text x="46.355" y="75.565" size="1.016" layer="21">BAT</text>
+<text x="46.482" y="41.529" size="1.016" layer="21">LOGR</text>
+<text x="49.149" y="45.085" size="1.016" layer="21" rot="R90">I2C NET</text>
+<text x="46.355" y="35.814" size="1.016" layer="21">SAT</text>
+<text x="46.228" y="30.226" size="1.016" layer="21">TEMP</text>
+<text x="46.482" y="26.289" size="1.016" layer="21">HEAT</text>
+<rectangle x1="35.179" y1="44.323" x2="47.752" y2="51.054" layer="21"/>
+<text x="48.641" y="56.642" size="1.016" layer="21" rot="R90">LEDS</text>
+<text x="43.688" y="68.961" size="2.1844" layer="21">+</text>
+<text x="43.561" y="38.481" size="2.1844" layer="21">+</text>
+<text x="43.688" y="32.258" size="2.1844" layer="21">+</text>
+<text x="43.688" y="23.241" size="2.1844" layer="21">+</text>
+<text x="44.196" y="63.627" size="2.1844" layer="21">-</text>
+<text x="43.688" y="77.851" size="2.1844" layer="21">+</text>
+<text x="6.35" y="79.502" size="1.016" layer="21">http://github.com/asfm-hlm-stemlab</text>
 </plain>
 <attributes>
@@
 <polygon width="0.1524" layer="1">
 <vertex x="0" y="91.44"/>
-<vertex x="0" y="15.24"/>
-<vertex x="49.53" y="15.24"/>
-<vertex x="49.53" y="91.44"/>
+<vertex x="-1.27" y="3.81"/>
+<vertex x="53.34" y="5.08"/>
+<vertex x="54.61" y="92.71"/>
 </polygon>
 <via x="4.191" y="86.868" extent="1-16" drill="3.17"/>
@@
 <polygon width="0.1524" layer="16">
 <vertex x="0" y="91.44"/>
-<vertex x="49.53" y="91.44"/>
-<vertex x="49.53" y="15.24"/>
-<vertex x="0" y="15.24"/>
+<vertex x="54.61" y="91.44"/>
+<vertex x="54.61" y="3.81"/>
+<vertex x="0" y="3.81"/>
 </polygon>
 <contactref element="R6" pad="1"/>
