File: NSP2D.sch (EAGLE design)
At the start: 21 parts, among them Q1 600mA/40V, Q2 IRF540

Commit message: Added missing pullup resistors to SCL SDA for I2C bus
Parts:
- added R6, R7: 4.5k, SparkFun-Passives:RESISTORPTH-1/6W
Connections:
- net SCL: now also R7.2
- net SDA: now also R6.2
- net V_BATT: now also R6.1, R7.1
Changed lines of the file:
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@@
 <part name="R4" library="SparkFun-Passives" deviceset="RESISTOR" device="PTH-1/6W" value="1K"/>
 <part name="LED3" library="SparkFun-Connectors" deviceset="CONN_02" device=""/>
+<part name="R6" library="SparkFun-Passives" deviceset="RESISTOR" device="PTH-1/6W" value="4.5k"/>
+<part name="R7" library="SparkFun-Passives" deviceset="RESISTOR" device="PTH-1/6W" value="4.5k"/>
+<part name="LI+7" library="SparkFun-PowerSymbols" deviceset="V_BATT" device=""/>
 </parts>
 <sheets>
@@
 <instance part="R4" gate="G$1" x="86.36" y="63.5" rot="R180"/>
 <instance part="LED3" gate="G$1" x="106.68" y="60.96" rot="MR0"/>
+<instance part="R6" gate="G$1" x="154.94" y="99.06" rot="R270"/>
+<instance part="R7" gate="G$1" x="162.56" y="99.06" rot="R270"/>
+<instance part="LI+7" gate="G$1" x="157.48" y="109.22"/>
 </instances>
 <busses>
@@
 <junction x="200.66" y="48.26"/>
 <pinref part="LI+6" gate="G$1" pin="V_BATT"/>
+</segment>
+<segment>
+<pinref part="R6" gate="G$1" pin="1"/>
+<pinref part="R7" gate="G$1" pin="1"/>
+<wire x1="154.94" y1="104.14" x2="157.48" y2="104.14" width="0.1524" layer="91"/>
+<wire x1="157.48" y1="104.14" x2="162.56" y2="104.14" width="0.1524" layer="91"/>
+<wire x1="157.48" y1="104.14" x2="157.48" y2="109.22" width="0.1524" layer="91"/>
+<junction x="157.48" y="104.14"/>
+<pinref part="LI+7" gate="G$1" pin="V_BATT"/>
 </segment>
 </net>
@@
 <wire x1="83.82" y1="38.1" x2="83.82" y2="30.48" width="0.1524" layer="91"/>
 <junction x="109.22" y="38.1"/>
+<label x="88.9" y="38.1" size="1.778" layer="95"/>
+</segment>
+<segment>
+<pinref part="R6" gate="G$1" pin="2"/>
+<wire x1="154.94" y1="93.98" x2="154.94" y2="88.9" width="0.1524" layer="91"/>
+<label x="147.32" y="88.9" size="1.778" layer="95"/>
 </segment>
 </net>
@@
 <wire x1="109.22" y1="35.56" x2="88.9" y2="35.56" width="0.1524" layer="91"/>
 <junction x="109.22" y="35.56"/>
-</segment>
-</net>
+<label x="91.44" y="33.02" size="1.778" layer="95"/>
+</segment>
+<segment>
+<pinref part="R7" gate="G$1" pin="2"/>
+<wire x1="162.56" y1="93.98" x2="162.56" y2="88.9" width="0.1524" layer="91"/>
+<label x="167.64" y="88.9" size="1.778" layer="95"/>
+</segment>
+</net>

Commit message: Added capacitor for batt source
Parts:
- added C1: 1mF, SparkFun-Capacitors:1000UF-RADIAL-5MM-25V-20%
- renumbered I2CX to I2C, I2CX1 to I2C1
Connections:
- net 3.3V: now also R6.1, R7.1
- net GND: now also C1.-
- net V_BATT: now also C1.+; no longer R6.1, R7.1
Other:
- moved on the sheet: R3
Changed lines of the file:
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@@
 <part name="BZR" library="SparkFun-Connectors" deviceset="CONN_02" device=""/>
 <part name="Q1" library="SparkFun-DiscreteSemi" deviceset="TRANS_NPN" device="-P2N2222A" value="600mA/40V"/>
-<part name="I2CX" library="SparkFun-Connectors" deviceset="CONN_04" device=""/>
+<part name="I2C" library="SparkFun-Connectors" deviceset="CONN_04" device=""/>
 <part name="LI+5" library="SparkFun-PowerSymbols" deviceset="V_BATT" device=""/>
-<part name="I2CX1" library="SparkFun-Connectors" deviceset="CONN_04" device=""/>
+<part name="I2C1" library="SparkFun-Connectors" deviceset="CONN_04" device=""/>
 <part name="TEMP" library="SparkFun-Connectors" deviceset="CONN_03" device="" value="455-1750-1-ND"/>
 <part name="SUPPLY1" library="SparkFun-PowerSymbols" deviceset="3.3V" device=""/>
@@
 <part name="R6" library="SparkFun-Passives" deviceset="RESISTOR" device="PTH-1/6W" value="4.5k"/>
 <part name="R7" library="SparkFun-Passives" deviceset="RESISTOR" device="PTH-1/6W" value="4.5k"/>
-<part name="LI+7" library="SparkFun-PowerSymbols" deviceset="V_BATT" device=""/>
+<part name="SUPPLY2" library="SparkFun-PowerSymbols" deviceset="3.3V" device=""/>
+<part name="C1" library="SparkFun-Capacitors" deviceset="1000UF" device="-RADIAL-5MM-25V-20%" value="1mF"/>
+<part name="GND10" library="supply1" library_urn="urn:adsk.eagle:library:371" deviceset="GND" device=""/>
 </parts>
 <sheets>
@@
 <instance part="LI+4" gate="G$1" x="149.86" y="68.58"/>
 <instance part="GND5" gate="1" x="152.4" y="48.26"/>
-<instance part="R3" gate="G$1" x="134.62" y="55.88" rot="R180"/>
+<instance part="R3" gate="G$1" x="129.54" y="55.88" rot="R180"/>
 <instance part="BZR" gate="G$1" x="160.02" y="60.96" rot="MR0"/>
 <instance part="Q1" gate="G$1" x="144.78" y="55.88"/>
-<instance part="I2CX" gate="G$1" x="129.54" y="38.1" rot="MR0"/>
+<instance part="I2C" gate="G$1" x="129.54" y="38.1" rot="MR0"/>
 <instance part="LI+5" gate="G$1" x="109.22" y="50.8"/>
-<instance part="I2CX1" gate="G$1" x="114.3" y="38.1" rot="MR0"/>
+<instance part="I2C1" gate="G$1" x="114.3" y="38.1" rot="MR0"/>
 <instance part="TEMP" gate="J$1" x="0" y="68.58"/>
 <instance part="SUPPLY1" gate="G$1" x="12.7" y="86.36"/>
@@
 <instance part="R6" gate="G$1" x="154.94" y="99.06" rot="R270"/>
 <instance part="R7" gate="G$1" x="162.56" y="99.06" rot="R270"/>
-<instance part="LI+7" gate="G$1" x="157.48" y="109.22"/>
+<instance part="SUPPLY2" gate="G$1" x="157.48" y="109.22"/>
+<instance part="C1" gate="G$1" x="127" y="88.9"/>
+<instance part="GND10" gate="1" x="142.24" y="78.74"/>
 </instances>
 <busses>
@@
 <wire x1="33.02" y1="86.36" x2="33.02" y2="93.98" width="0.1524" layer="91"/>
 </segment>
+<segment>
+<pinref part="R6" gate="G$1" pin="1"/>
+<pinref part="R7" gate="G$1" pin="1"/>
+<wire x1="154.94" y1="104.14" x2="157.48" y2="104.14" width="0.1524" layer="91"/>
+<wire x1="157.48" y1="104.14" x2="162.56" y2="104.14" width="0.1524" layer="91"/>
+<wire x1="157.48" y1="104.14" x2="157.48" y2="109.22" width="0.1524" layer="91"/>
+<junction x="157.48" y="104.14"/>
+<pinref part="SUPPLY2" gate="G$1" pin="3.3V"/>
+</segment>
 </net>
 <net name="V_BATT" class="0">
@@
 <wire x1="109.22" y1="96.52" x2="109.22" y2="91.44" width="0.1524" layer="91"/>
 <wire x1="119.38" y1="91.44" x2="109.22" y2="91.44" width="0.1524" layer="91"/>
+<pinref part="C1" gate="G$1" pin="+"/>
+<wire x1="127" y1="91.44" x2="119.38" y2="91.44" width="0.1524" layer="91"/>
+<junction x="119.38" y="91.44"/>
 </segment>
 <segment>
@@
 <segment>
 <pinref part="LI+5" gate="G$1" pin="V_BATT"/>
-<pinref part="I2CX1" gate="G$1" pin="4"/>
+<pinref part="I2C1" gate="G$1" pin="4"/>
 <wire x1="109.22" y1="50.8" x2="109.22" y2="48.26" width="0.1524" layer="91"/>
-<pinref part="I2CX" gate="G$1" pin="4"/>
+<pinref part="I2C" gate="G$1" pin="4"/>
 <wire x1="109.22" y1="48.26" x2="109.22" y2="43.18" width="0.1524" layer="91"/>
 <wire x1="124.46" y1="48.26" x2="124.46" y2="43.18" width="0.1524" layer="91"/>
@@
 <pinref part="LI+6" gate="G$1" pin="V_BATT"/>
 </segment>
-<segment>
-<pinref part="R6" gate="G$1" pin="1"/>
-<pinref part="R7" gate="G$1" pin="1"/>
-<wire x1="154.94" y1="104.14" x2="157.48" y2="104.14" width="0.1524" layer="91"/>
-<wire x1="157.48" y1="104.14" x2="162.56" y2="104.14" width="0.1524" layer="91"/>
-<wire x1="157.48" y1="104.14" x2="157.48" y2="109.22" width="0.1524" layer="91"/>
-<junction x="157.48" y="104.14"/>
-<pinref part="LI+7" gate="G$1" pin="V_BATT"/>
-</segment>
 </net>
 <net name="UART5_RX" class="0">
@@
 <segment>
 <pinref part="GND2" gate="1" pin="GND"/>
-<pinref part="I2CX" gate="G$1" pin="3"/>
-<pinref part="I2CX1" gate="G$1" pin="3"/>
+<pinref part="I2C" gate="G$1" pin="3"/>
+<pinref part="I2C1" gate="G$1" pin="3"/>
 <wire x1="109.22" y1="40.64" x2="124.46" y2="40.64" width="0.1524" layer="91"/>
 <wire x1="109.22" y1="40.64" x2="104.14" y2="40.64" width="0.1524" layer="91"/>
@@
 <junction x="96.52" y="71.12"/>
 </segment>
+<segment>
+<pinref part="C1" gate="G$1" pin="-"/>
+<wire x1="127" y1="83.82" x2="142.24" y2="83.82" width="0.1524" layer="91"/>
+<wire x1="142.24" y1="83.82" x2="142.24" y2="81.28" width="0.1524" layer="91"/>
+<pinref part="GND10" gate="1" pin="GND"/>
+</segment>
 </net>
 <net name="IRWKP" class="0">
@@
 <net name="SDA" class="0">
 <segment>
-<pinref part="I2CX1" gate="G$1" pin="2"/>
-<pinref part="I2CX" gate="G$1" pin="2"/>
+<pinref part="I2C1" gate="G$1" pin="2"/>
+<pinref part="I2C" gate="G$1" pin="2"/>
 <wire x1="109.22" y1="38.1" x2="124.46" y2="38.1" width="0.1524" layer="91"/>
 <pinref part="MCU" gate="G$1" pin="C5"/>
@@
 <wire x1="129.54" y1="25.4" x2="129.54" y2="27.94" width="0.1524" layer="91"/>
 <wire x1="129.54" y1="27.94" x2="91.44" y2="27.94" width="0.1524" layer="91"/>
-</segment>
-</net>
-<net name="N$6" class="0">
-<segment>
-<pinref part="MCU" gate="G$1" pin="D4"/>
-<wire x1="76.2" y1="55.88" x2="129.54" y2="55.88" width="0.1524" layer="91"/>
-<pinref part="R3" gate="G$1" pin="2"/>
-</segment>
-</net>
-<net name="N$10" class="0">
-<segment>
-<pinref part="R3" gate="G$1" pin="1"/>
-<wire x1="139.7" y1="55.88" x2="142.24" y2="55.88" width="0.1524" layer="91"/>
-<pinref part="Q1" gate="G$1" pin="B"/>
 </segment>
 </net>
@@
 <net name="SCL" class="0">
 <segment>
-<pinref part="I2CX" gate="G$1" pin="1"/>
-<pinref part="I2CX1" gate="G$1" pin="1"/>
+<pinref part="I2C" gate="G$1" pin="1"/>
+<pinref part="I2C1" gate="G$1" pin="1"/>
 <wire x1="124.46" y1="35.56" x2="109.22" y2="35.56" width="0.1524" layer="91"/>
 <wire x1="88.9" y1="25.4" x2="88.9" y2="35.56" width="0.1524" layer="91"/>
@@
 </segment>
 </net>
+<net name="N$4" class="0">
+<segment>
+<pinref part="R3" gate="G$1" pin="1"/>
+<pinref part="Q1" gate="G$1" pin="B"/>
+<wire x1="134.62" y1="55.88" x2="142.24" y2="55.88" width="0.1524" layer="91"/>
+</segment>
+</net>
+<net name="N$5" class="0">
+<segment>
+<pinref part="R3" gate="G$1" pin="2"/>
+<pinref part="MCU" gate="G$1" pin="D4"/>
+<wire x1="124.46" y1="55.88" x2="76.2" y2="55.88" width="0.1524" layer="91"/>
+</segment>
+</net>
