File: HLM1_Outsourced.sch (EAGLE design)
At the start: 24 parts, among them Q1 600mA/40V, Q2 IRF540

Commit message: Added onboard level shifter to outsourced design and other improvements
Parts:
- removed IRIDIUM: (no value), SparkFun-Connectors:CONN_05
- removed Q2: IRF540, transistor-fet:IRF540
- added 3V3, SW1: (no value), SparkFun-Connectors:CONN_02
- added B1: SPARKFUN_LOGIC_LEVEL_CONVERTER, SparkFun-Boards:SPARKFUN_LOGIC_LEVEL_CONVERTER
- added J3: (no value), SparkFun-Connectors:CONN_06SILK_FEMALE_PTH
- added Q3: 60V/32A/35mΩ, SparkFun-DiscreteSemi:MOSFET-NCH-FQP30N06L
Connections:
- removed net UART5_RX: IRIDIUM.1, MCU.C0
- new net 5VREF: B1.HV, J3.1
- new net N$10: B1.HV_TXO_1, J3.3
- new net N$15: MCU.A5, SW1.1
- new net N$6: B1.LV_TXI_1, MCU.C1
- new net N$7: B1.LV_RXO_1, MCU.C0
- net 3.3V: now also 3V3.2, B1.LV, SW1.2
- net D3: now also Q3.G; no longer Q2.G
- net GND: now also 3V3.1, B1.GND, B1.GND@2, J3.5, Q3.S; no longer IRIDIUM.4, Q2.S
- net IRWKP: now also J3.4; no longer IRIDIUM.3
- net N$11: now also Q3.D; no longer Q2.D
- net N$14: now also B1.HV_RXI_1, J3.2; no longer IRIDIUM.2, MCU.C1
- net V_BATT: now also J3.6; no longer IRIDIUM.5

Commit message: Added onboard SD CARD + Sonar Port for touchdown detection
Parts:
- added ITEMP: (no value), SparkFun-Sensors:TMP36GT9
- added JP2: (no value), SparkFun-Connectors:M06NO_SILK_FEMALE_PTH
- added SONAR: 455-1750-1-ND, SparkFun-Connectors:CONN_03
- renumbered TEMP to XTEMP
Connections:
- new net N$17: MCU.A1, SONAR.1
- new net N$21: ITEMP.VOUT, MCU.A0
- net 3.3V: now also ITEMP.VCC, JP2.3, SONAR.3
- net GND: now also ITEMP.GND, JP2.1, JP2.2, SONAR.2
- net UART4_RX: now also JP2.4
- net UART4_TX: now also JP2.5
Other:
- moved on the sheet: LOGR
Changed lines of the file:
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@@
 </variantdefs>
 <classes>
-<class number="0" name="default" width="0" drill="0">
+<class number="0" name="default" width="0.1778" drill="0">
+</class>
+<class number="1" name="vcc" width="0.2032" drill="0">
 </class>
 </classes>
@@
 <part name="LI+5" library="SparkFun-PowerSymbols" deviceset="V_BATT" device=""/>
 <part name="I2C1" library="SparkFun-Connectors" deviceset="CONN_04" device=""/>
-<part name="TEMP" library="SparkFun-Connectors" deviceset="CONN_03" device="" value="455-1750-1-ND"/>
+<part name="XTEMP" library="SparkFun-Connectors" deviceset="CONN_03" device="" value="455-1750-1-ND"/>
 <part name="SUPPLY1" library="SparkFun-PowerSymbols" deviceset="3.3V" device=""/>
 <part name="GND6" library="supply1" library_urn="urn:adsk.eagle:library:371" deviceset="GND" device=""/>
@@
 <part name="SW1" library="SparkFun-Connectors" deviceset="CONN_02" device=""/>
 <part name="SUPPLY7" library="SparkFun-PowerSymbols" deviceset="3.3V" device=""/>
+<part name="SONAR" library="SparkFun-Connectors" deviceset="CONN_03" device="" value="455-1750-1-ND"/>
+<part name="SUPPLY8" library="SparkFun-PowerSymbols" deviceset="3.3V" device=""/>
+<part name="GND13" library="supply1" library_urn="urn:adsk.eagle:library:371" deviceset="GND" device=""/>
+<part name="ITEMP" library="SparkFun-Sensors" deviceset="TMP36" device="GT9"/>
+<part name="GND14" library="supply1" library_urn="urn:adsk.eagle:library:371" deviceset="GND" device=""/>
+<part name="SUPPLY9" library="SparkFun-PowerSymbols" deviceset="3.3V" device=""/>
+<part name="GND21" library="SparkFun" deviceset="GND" device=""/>
+<part name="JP2" library="SparkFun-Connectors" deviceset="M06" device="NO_SILK_FEMALE_PTH"/>
 </parts>
 <sheets>
@@
 <instance part="GND3" gate="1" x="121.92" y="66.04"/>
 <instance part="LI+2" gate="G$1" x="121.92" y="73.66"/>
-<instance part="LOGR" gate="G$1" x="149.86" y="25.4" rot="MR0"/>
+<instance part="LOGR" gate="G$1" x="147.32" y="25.4" rot="MR0"/>
 <instance part="GND4" gate="1" x="134.62" y="15.24"/>
 <instance part="LI+3" gate="G$1" x="139.7" y="38.1"/>
@@
 <instance part="LI+5" gate="G$1" x="109.22" y="50.8"/>
 <instance part="I2C1" gate="G$1" x="114.3" y="38.1" rot="MR0"/>
-<instance part="TEMP" gate="J$1" x="0" y="68.58"/>
+<instance part="XTEMP" gate="J$1" x="0" y="68.58"/>
 <instance part="SUPPLY1" gate="G$1" x="12.7" y="86.36"/>
 <instance part="GND6" gate="1" x="12.7" y="53.34"/>
@@
 <instance part="SW1" gate="G$1" x="27.94" y="53.34"/>
 <instance part="SUPPLY7" gate="G$1" x="25.4" y="68.58"/>
+<instance part="SONAR" gate="J$1" x="20.32" y="35.56"/>
+<instance part="SUPPLY8" gate="G$1" x="30.48" y="40.64"/>
+<instance part="GND13" gate="1" x="30.48" y="22.86"/>
+<instance part="ITEMP" gate="G$1" x="17.78" y="10.16"/>
+<instance part="GND14" gate="1" x="5.08" y="0"/>
+<instance part="SUPPLY9" gate="G$1" x="5.08" y="20.32"/>
+<instance part="GND21" gate="1" x="172.72" y="17.78"/>
+<instance part="JP2" gate="G$1" x="160.02" y="27.94"/>
 </instances>
 <busses>
@@
 </segment>
 <segment>
-<pinref part="TEMP" gate="J$1" pin="3"/>
+<pinref part="XTEMP" gate="J$1" pin="3"/>
 <wire x1="7.62" y1="71.12" x2="12.7" y2="71.12" width="0.1524" layer="91"/>
 <pinref part="SUPPLY1" gate="G$1" pin="3.3V"/>
@@
 <wire x1="35.56" y1="60.96" x2="25.4" y2="60.96" width="0.1524" layer="91"/>
 <wire x1="25.4" y1="60.96" x2="25.4" y2="68.58" width="0.1524" layer="91"/>
+</segment>
+<segment>
+<pinref part="SONAR" gate="J$1" pin="3"/>
+<wire x1="27.94" y1="38.1" x2="30.48" y2="38.1" width="0.1524" layer="91"/>
+<pinref part="SUPPLY8" gate="G$1" pin="3.3V"/>
+<wire x1="30.48" y1="38.1" x2="30.48" y2="40.64" width="0.1524" layer="91"/>
+</segment>
+<segment>
+<pinref part="ITEMP" gate="G$1" pin="VCC"/>
+<wire x1="10.16" y1="12.7" x2="5.08" y2="12.7" width="0.1524" layer="91"/>
+<wire x1="5.08" y1="12.7" x2="5.08" y2="20.32" width="0.1524" layer="91"/>
+<pinref part="SUPPLY9" gate="G$1" pin="3.3V"/>
+</segment>
+<segment>
+<pinref part="JP2" gate="G$1" pin="3"/>
+<wire x1="165.1" y1="27.94" x2="167.64" y2="27.94" width="0.1524" layer="91"/>
+<label x="168.148" y="26.924" size="1.778" layer="95"/>
 </segment>
 </net>
@@
 <wire x1="139.7" y1="38.1" x2="139.7" y2="30.48" width="0.1524" layer="91"/>
 <pinref part="LOGR" gate="G$1" pin="4"/>
-<wire x1="139.7" y1="30.48" x2="144.78" y2="30.48" width="0.1524" layer="91"/>
+<wire x1="139.7" y1="30.48" x2="142.24" y2="30.48" width="0.1524" layer="91"/>
 </segment>
 <segment>
@@
 <pinref part="GND4" gate="1" pin="GND"/>
 <pinref part="LOGR" gate="G$1" pin="3"/>
-<wire x1="144.78" y1="27.94" x2="134.62" y2="27.94" width="0.1524" layer="91"/>
+<wire x1="142.24" y1="27.94" x2="134.62" y2="27.94" width="0.1524" layer="91"/>
 <wire x1="134.62" y1="27.94" x2="134.62" y2="17.78" width="0.1524" layer="91"/>
 </segment>
@@
 <pinref part="GND6" gate="1" pin="GND"/>
 <wire x1="12.7" y1="68.58" x2="12.7" y2="55.88" width="0.1524" layer="91"/>
-<pinref part="TEMP" gate="J$1" pin="2"/>
+<pinref part="XTEMP" gate="J$1" pin="2"/>
 <wire x1="7.62" y1="68.58" x2="12.7" y2="68.58" width="0.1524" layer="91"/>
 </segment>
@@
 <wire x1="170.18" y1="71.12" x2="170.18" y2="68.58" width="0.1524" layer="91"/>
 </segment>
+<segment>
+<pinref part="SONAR" gate="J$1" pin="2"/>
+<wire x1="27.94" y1="35.56" x2="30.48" y2="35.56" width="0.1524" layer="91"/>
+<wire x1="30.48" y1="35.56" x2="30.48" y2="25.4" width="0.1524" layer="91"/>
+<pinref part="GND13" gate="1" pin="GND"/>
+</segment>
+<segment>
+<pinref part="ITEMP" gate="G$1" pin="GND"/>
+<wire x1="10.16" y1="7.62" x2="5.08" y2="7.62" width="0.1524" layer="91"/>
+<wire x1="5.08" y1="7.62" x2="5.08" y2="2.54" width="0.1524" layer="91"/>
+<pinref part="GND14" gate="1" pin="GND"/>
+</segment>
+<segment>
+<wire x1="172.72" y1="22.86" x2="172.72" y2="20.32" width="0.1524" layer="91"/>
+<pinref part="GND21" gate="1" pin="GND"/>
+<wire x1="165.1" y1="25.4" x2="172.72" y2="25.4" width="0.1524" layer="91"/>
+<wire x1="172.72" y1="25.4" x2="172.72" y2="22.86" width="0.1524" layer="91"/>
+<wire x1="165.1" y1="22.86" x2="172.72" y2="22.86" width="0.1524" layer="91"/>
+<junction x="172.72" y="22.86"/>
+<pinref part="JP2" gate="G$1" pin="1"/>
+<pinref part="JP2" gate="G$1" pin="2"/>
+</segment>
 </net>
 <net name="IRWKP" class="0">
@@
 <wire x1="127" y1="25.4" x2="127" y2="22.86" width="0.1524" layer="91"/>
 <pinref part="LOGR" gate="G$1" pin="1"/>
-<wire x1="127" y1="22.86" x2="144.78" y2="22.86" width="0.1524" layer="91"/>
+<wire x1="127" y1="22.86" x2="142.24" y2="22.86" width="0.1524" layer="91"/>
+<label x="129.54" y="22.86" size="1.778" layer="95" rot="R180"/>
+</segment>
+<segment>
+<wire x1="165.1" y1="30.48" x2="167.64" y2="30.48" width="0.1524" layer="91"/>
+<label x="167.64" y="30.48" size="1.27" layer="95" rot="MR180" xref="yes"/>
+<pinref part="JP2" gate="G$1" pin="4"/>
 </segment>
 </net>
@@
 <wire x1="91.44" y1="20.32" x2="76.2" y2="20.32" width="0.1524" layer="91"/>
 <pinref part="LOGR" gate="G$1" pin="2"/>
-<wire x1="144.78" y1="25.4" x2="129.54" y2="25.4" width="0.1524" layer="91"/>
+<wire x1="142.24" y1="25.4" x2="129.54" y2="25.4" width="0.1524" layer="91"/>
 <wire x1="129.54" y1="25.4" x2="129.54" y2="27.94" width="0.1524" layer="91"/>
 <wire x1="129.54" y1="27.94" x2="91.44" y2="27.94" width="0.1524" layer="91"/>
+<label x="129.54" y="30.48" size="1.778" layer="95" rot="R180"/>
+</segment>
+<segment>
+<wire x1="165.1" y1="33.02" x2="167.64" y2="33.02" width="0.1524" layer="91"/>
+<label x="167.64" y="33.02" size="1.27" layer="95" rot="MR180" xref="yes"/>
+<pinref part="JP2" gate="G$1" pin="5"/>
 </segment>
 </net>
@@
 <pinref part="MCU" gate="G$1" pin="DAC"/>
 <wire x1="40.64" y1="66.04" x2="7.62" y2="66.04" width="0.1524" layer="91"/>
-<pinref part="TEMP" gate="J$1" pin="1"/>
+<pinref part="XTEMP" gate="J$1" pin="1"/>
 </segment>
 </net>
@@
 </segment>
 </net>
+<net name="N$17" class="0">
+<segment>
+<pinref part="SONAR" gate="J$1" pin="1"/>
+<wire x1="33.02" y1="33.02" x2="27.94" y2="33.02" width="0.1524" layer="91"/>
+<pinref part="MCU" gate="G$1" pin="A1"/>
+<wire x1="40.64" y1="40.64" x2="33.02" y2="40.64" width="0.1524" layer="91"/>
+<wire x1="33.02" y1="40.64" x2="33.02" y2="33.02" width="0.1524" layer="91"/>
+</segment>
+</net>
+<net name="N$21" class="0">
+<segment>
+<pinref part="MCU" gate="G$1" pin="A0"/>
+<wire x1="40.64" y1="35.56" x2="35.56" y2="35.56" width="0.1524" layer="91"/>
+<wire x1="35.56" y1="35.56" x2="35.56" y2="10.16" width="0.1524" layer="91"/>
+<wire x1="35.56" y1="10.16" x2="25.4" y2="10.16" width="0.1524" layer="91"/>
+<pinref part="ITEMP" gate="G$1" pin="VOUT"/>
+</segment>
+</net>

Commit message: Improved design and labels
Parts:
- B1: value SPARKFUN_LOGIC_LEVEL_CONVERTER -> LOGIC LEVEL SHIFTER
- Q3: value 60V/32A/35mΩ -> MOSFET
- SONAR: value 455-1750-1-ND -> SONAR
- renumbered HEATPADS to HEAT, J3 to SATCOM, JP2 to SD
Changed lines of the file:
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@@
 <part name="SUPPLY1" library="SparkFun-PowerSymbols" deviceset="3.3V" device=""/>
 <part name="GND6" library="supply1" library_urn="urn:adsk.eagle:library:371" deviceset="GND" device=""/>
-<part name="HEATPADS" library="SparkFun-Connectors" deviceset="CONN_04" device=""/>
+<part name="HEAT" library="SparkFun-Connectors" deviceset="CONN_04" device=""/>
 <part name="GND7" library="supply1" library_urn="urn:adsk.eagle:library:371" deviceset="GND" device=""/>
 <part name="LI+6" library="SparkFun-PowerSymbols" deviceset="V_BATT" device=""/>
@@
 <part name="C1" library="SparkFun-Capacitors" deviceset="1000UF" device="-RADIAL-5MM-25V-20%" value="1mF"/>
 <part name="GND10" library="supply1" library_urn="urn:adsk.eagle:library:371" deviceset="GND" device=""/>
-<part name="B1" library="SparkFun-Boards" deviceset="SPARKFUN_LOGIC_LEVEL_CONVERTER" device=""/>
+<part name="B1" library="SparkFun-Boards" deviceset="SPARKFUN_LOGIC_LEVEL_CONVERTER" device="" value="LOGIC LEVEL SHIFTER"/>
 <part name="GND11" library="supply1" library_urn="urn:adsk.eagle:library:371" deviceset="GND" device=""/>
 <part name="SUPPLY5" library="SparkFun-PowerSymbols" deviceset="3.3V" device=""/>
-<part name="J3" library="SparkFun-Connectors" deviceset="CONN_06" device="SILK_FEMALE_PTH"/>
+<part name="SATCOM" library="SparkFun-Connectors" deviceset="CONN_06" device="SILK_FEMALE_PTH"/>
 <part name="3V3" library="SparkFun-Connectors" deviceset="CONN_02" device=""/>
 <part name="GND12" library="supply1" library_urn="urn:adsk.eagle:library:371" deviceset="GND" device=""/>
 <part name="SUPPLY6" library="SparkFun-PowerSymbols" deviceset="3.3V" device=""/>
-<part name="Q3" library="SparkFun-DiscreteSemi" deviceset="MOSFET-NCH" device="-FQP30N06L" value="60V/32A/35mΩ"/>
+<part name="Q3" library="SparkFun-DiscreteSemi" deviceset="MOSFET-NCH" device="-FQP30N06L" value="MOSFET"/>
 <part name="SW1" library="SparkFun-Connectors" deviceset="CONN_02" device=""/>
 <part name="SUPPLY7" library="SparkFun-PowerSymbols" deviceset="3.3V" device=""/>
-<part name="SONAR" library="SparkFun-Connectors" deviceset="CONN_03" device="" value="455-1750-1-ND"/>
+<part name="SONAR" library="SparkFun-Connectors" deviceset="CONN_03" device="" value="SONAR"/>
 <part name="SUPPLY8" library="SparkFun-PowerSymbols" deviceset="3.3V" device=""/>
 <part name="GND13" library="supply1" library_urn="urn:adsk.eagle:library:371" deviceset="GND" device=""/>
@@
 <part name="SUPPLY9" library="SparkFun-PowerSymbols" deviceset="3.3V" device=""/>
 <part name="GND21" library="SparkFun" deviceset="GND" device=""/>
-<part name="JP2" library="SparkFun-Connectors" deviceset="M06" device="NO_SILK_FEMALE_PTH"/>
+<part name="SD" library="SparkFun-Connectors" deviceset="M06" device="NO_SILK_FEMALE_PTH"/>
 </parts>
 <sheets>
@@
 <instance part="SUPPLY1" gate="G$1" x="12.7" y="86.36"/>
 <instance part="GND6" gate="1" x="12.7" y="53.34"/>
-<instance part="HEATPADS" gate="G$1" x="210.82" y="43.18" rot="MR0"/>
+<instance part="HEAT" gate="G$1" x="210.82" y="43.18" rot="MR0"/>
 <instance part="GND7" gate="1" x="193.04" y="22.86"/>
 <instance part="LI+6" gate="G$1" x="200.66" y="55.88"/>
@@
 <instance part="GND11" gate="1" x="99.06" y="-27.94"/>
 <instance part="SUPPLY5" gate="G$1" x="63.5" y="-7.62"/>
-<instance part="J3" gate="G$1" x="177.8" y="5.08" rot="MR0"/>
+<instance part="SATCOM" gate="G$1" x="177.8" y="5.08" rot="MR0"/>
 <instance part="3V3" gate="G$1" x="182.88" y="71.12" rot="MR0"/>
 <instance part="GND12" gate="1" x="170.18" y="66.04"/>
@@
 <instance part="SUPPLY9" gate="G$1" x="5.08" y="20.32"/>
 <instance part="GND21" gate="1" x="172.72" y="17.78"/>
-<instance part="JP2" gate="G$1" x="160.02" y="27.94"/>
+<instance part="SD" gate="G$1" x="160.02" y="27.94"/>
 </instances>
 <busses>
@@
 </segment>
 <segment>
-<pinref part="JP2" gate="G$1" pin="3"/>
+<pinref part="SD" gate="G$1" pin="3"/>
 <wire x1="165.1" y1="27.94" x2="167.64" y2="27.94" width="0.1524" layer="91"/>
 <label x="168.148" y="26.924" size="1.778" layer="95"/>
@@
 <wire x1="104.14" y1="20.32" x2="104.14" y2="12.7" width="0.1524" layer="91"/>
 <wire x1="172.72" y1="12.7" x2="104.14" y2="12.7" width="0.1524" layer="91"/>
-<pinref part="J3" gate="G$1" pin="6"/>
+<pinref part="SATCOM" gate="G$1" pin="6"/>
 </segment>
 <segment>
@@
 </segment>
 <segment>
-<pinref part="HEATPADS" gate="G$1" pin="4"/>
+<pinref part="HEAT" gate="G$1" pin="4"/>
 <wire x1="205.74" y1="48.26" x2="200.66" y2="48.26" width="0.1524" layer="91"/>
 <wire x1="200.66" y1="48.26" x2="200.66" y2="43.18" width="0.1524" layer="91"/>
-<pinref part="HEATPADS" gate="G$1" pin="2"/>
+<pinref part="HEAT" gate="G$1" pin="2"/>
 <wire x1="200.66" y1="43.18" x2="205.74" y2="43.18" width="0.1524" layer="91"/>
 <wire x1="200.66" y1="48.26" x2="200.66" y2="55.88" width="0.1524" layer="91"/>
@@
 <wire x1="172.72" y1="10.16" x2="104.14" y2="10.16" width="0.1524" layer="91"/>
 <wire x1="104.14" y1="10.16" x2="104.14" y2="5.08" width="0.1524" layer="91"/>
-<pinref part="J3" gate="G$1" pin="5"/>
+<pinref part="SATCOM" gate="G$1" pin="5"/>
 </segment>
 <segment>
@@
 <wire x1="165.1" y1="22.86" x2="172.72" y2="22.86" width="0.1524" layer="91"/>
 <junction x="172.72" y="22.86"/>
-<pinref part="JP2" gate="G$1" pin="1"/>
-<pinref part="JP2" gate="G$1" pin="2"/>
+<pinref part="SD" gate="G$1" pin="1"/>
+<pinref part="SD" gate="G$1" pin="2"/>
 </segment>
 </net>
@@
 <wire x1="99.06" y1="45.72" x2="99.06" y2="7.62" width="0.1524" layer="91"/>
 <wire x1="99.06" y1="7.62" x2="172.72" y2="7.62" width="0.1524" layer="91"/>
-<pinref part="J3" gate="G$1" pin="4"/>
+<pinref part="SATCOM" gate="G$1" pin="4"/>
 </segment>
 </net>
@@
 <wire x1="165.1" y1="30.48" x2="167.64" y2="30.48" width="0.1524" layer="91"/>
 <label x="167.64" y="30.48" size="1.27" layer="95" rot="MR180" xref="yes"/>
-<pinref part="JP2" gate="G$1" pin="4"/>
+<pinref part="SD" gate="G$1" pin="4"/>
 </segment>
 </net>
@@
 <wire x1="165.1" y1="33.02" x2="167.64" y2="33.02" width="0.1524" layer="91"/>
 <label x="167.64" y="33.02" size="1.27" layer="95" rot="MR180" xref="yes"/>
-<pinref part="JP2" gate="G$1" pin="5"/>
+<pinref part="SD" gate="G$1" pin="5"/>
 </segment>
 </net>
@@
 <wire x1="190.5" y1="45.72" x2="198.12" y2="45.72" width="0.1524" layer="91"/>
 <wire x1="198.12" y1="45.72" x2="198.12" y2="40.64" width="0.1524" layer="91"/>
-<pinref part="HEATPADS" gate="G$1" pin="1"/>
+<pinref part="HEAT" gate="G$1" pin="1"/>
 <wire x1="198.12" y1="40.64" x2="205.74" y2="40.64" width="0.1524" layer="91"/>
-<pinref part="HEATPADS" gate="G$1" pin="3"/>
+<pinref part="HEAT" gate="G$1" pin="3"/>
 <wire x1="198.12" y1="45.72" x2="205.74" y2="45.72" width="0.1524" layer="91"/>
 <junction x="198.12" y="45.72"/>
@@
 <wire x1="124.46" y1="-5.08" x2="124.46" y2="5.08" width="0.1524" layer="91"/>
 <wire x1="124.46" y1="5.08" x2="172.72" y2="5.08" width="0.1524" layer="91"/>
-<pinref part="J3" gate="G$1" pin="3"/>
+<pinref part="SATCOM" gate="G$1" pin="3"/>
 </segment>
 </net>
@@
 <pinref part="B1" gate="G$1" pin="HV_RXI_1"/>
 <wire x1="127" y1="-7.62" x2="116.84" y2="-7.62" width="0.1524" layer="91"/>
-<pinref part="J3" gate="G$1" pin="2"/>
+<pinref part="SATCOM" gate="G$1" pin="2"/>
 </segment>
 </net>
@@
 <wire x1="160.02" y1="-10.16" x2="160.02" y2="0" width="0.1524" layer="91"/>
 <label x="162.56" y="-10.16" size="1.778" layer="95"/>
-<pinref part="J3" gate="G$1" pin="1"/>
+<pinref part="SATCOM" gate="G$1" pin="1"/>
 <wire x1="172.72" y1="0" x2="160.02" y2="0" width="0.1524" layer="91"/>
 </segment>

Commit message: Minor Updates
Connections:
- net N$12 renamed RX
- net N$2 renamed TX
Changed lines of the file:
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@@
 </segment>
 </net>
-<net name="N$12" class="0">
+<net name="RX" class="0">
 <segment>
 <pinref part="MCU" gate="G$1" pin="RX"/>
@@
 </segment>
 </net>
-<net name="N$2" class="0">
+<net name="TX" class="0">
 <segment>
 <pinref part="MCU" gate="G$1" pin="TX"/>
