File: HLM1_Outsourced_V2.sch (EAGLE design)
At the start: 33 parts, among them Q1 600mA/40V, Q2 MOSFET, Q3 MOSFET, SW1 SW1

Commit message: Updated flight board to add XBee radio
Parts:
- removed JP1: (no value), SparkFun-RF:XBEE
- added XBEE: RAD, SparkFun-RF:XBEELONGPAD
- renumbered SONAR to SN
Connections:
- removed net N$12: GPS.2, MCU.A3
- removed net N$2: GPS.1, MCU.A2
- removed net N$20: JP1.DIN, MCU.TX
- removed net N$22: JP1.DOUT, MCU.RX
- removed net X_RESET: JP1.RESET, MCU.B0
- removed net X_RSSI: JP1.RSSI, MCU.B3
- removed net X_RTS: JP1.RTS, MCU.B1
- new net GPSRX: GPS.1, MCU.RX
- new net GPSTX: GPS.2, MCU.TX
- new net XBEE_DIN: MCU.A3, XBEE.DIN
- new net XBEE_DOUT: MCU.A2, XBEE.DOUT
- net 3.3V: now also XBEE.VDD; no longer JP1.VDD
- net GND: now also XBEE.GND; no longer JP1.GND
Other:
- moved on the sheet: GPS, XTEMP
